File: KiCad/flight_controller_pcb.kicad_pcb (KiCad board)
At the start: 2 copper layers, 44 x 48 mm, 43 parts, among them J2 Conn_01x04_Pin, J3 Conn_01x03_Pin, J4 Conn_01x03_Pin, J5 Conn_01x03_Pin, J6 Conn_01x03_Pin, J7 USB3_B_Micro, SW1 SW_SPDT, U1 STM32F405RGTx, U2 AMS1117-3.3, U4 ICM-20602, U5 BMP280, Y1 16Mhz

Commit message: Improve project documentation and structure
Parts:
- moved SW1 2.50 mm to (101.5, 71.0)
- moved J7 2.50 mm to (130.0, 62.3)
Routing:
- net Net-(SW1-B): track 5.05 -> 8.05 mm
- net /USB_D-: track 16.8 -> 19.3 mm
- net /USB_D+: track 16.0 -> 18.5 mm
- net VBUS: track 76.3 -> 78.8 mm
- net +3.3V: track 132.3 -> 134.8 mm
- net GND: track 91.0 -> 90.9 mm, vias 21 -> 22
Changed lines of the file:
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@@
 		(filling no)
 		(pcbplotparams
-			(layerselection 0x00000000_00000000_55555555_5755f5ff)
+			(layerselection 0x00000000_00000000_55555555_575555ff)
 			(plot_on_all_layers_selection 0x00000000_00000000_00000000_00000000)
 			(disableapertmacros no)
@@
 			(outputformat 1)
 			(mirror no)
-			(drillshape 1)
+			(drillshape 0)
 			(scaleselection 1)
 			(outputdirectory "")
@@
 	(footprint "Button_Switch_SMD:SW_SPDT_PCM12"
 		(layer "F.Cu")
-		(at 104 71 -90)
+		(at 101.5 71 -90)
 		(descr "Ultraminiature Surface Mount Slide Switch, right-angle, https://www.ckswitches.com/media/1424/pcm.pdf")
 		(property "Reference" "SW1"
@@
 		(duplicate_pad_numbers_are_jumpers no)
 		(fp_line
-			(start -2.85 1.73)
-			(end 2.85 1.73)
-			(stroke
-				(width 0.12)
-				(type solid)
-			)
-			(layer "F.SilkS")
-		)
-		(fp_line
 			(start 3.45 0.72)
 			(end 3.45 -0.07)
@@
 	(footprint "Connector_USB:USB_Micro-B_Wuerth_629105150521"
 		(layer "F.Cu")
-		(at 130.005 64.755 180)
+		(at 130.005 62.255 180)
 		(descr "USB Micro-B receptacle, http://www.mouser.com/ds/2/445/629105150521-469306.pdf")
 		(tags "usb micro receptacle")
@@
 	)
 	(segment
+		(start 105.875 73.25)
+		(end 102.93 73.25)
+		(width 0.5)
+		(layer "F.Cu")
+		(net "+3.3V")
+	)
+	(segment
 		(start 132.85 78)
 		(end 132.85 74.35)
@@
 	)
 	(segment
+		(start 106 73.375)
+		(end 108.5 73.375)
+		(width 0.5)
+		(layer "F.Cu")
+		(net "+3.3V")
+	)
+	(segment
 		(start 126.725 87.225)
 		(end 123 87.225)
@@
 	)
 	(segment
-		(start 105.555 73.375)
-		(end 108.5 73.375)
-		(width 0.5)
-		(layer "F.Cu")
-		(net "+3.3V")
-	)
-	(segment
 		(start 115.7 65.7)
 		(end 115.775 65.7)
@@
 	)
 	(segment
-		(start 105.43 73.25)
-		(end 105.555 73.375)
-		(width 0.5)
-		(layer "F.Cu")
-		(net "+3.3V")
-	)
-	(segment
 		(start 120.15 87.590256)
 		(end 120.15 88.709744)
@@
 	)
 	(segment
+		(start 106 73.375)
+		(end 105.875 73.25)
+		(width 0.5)
+		(layer "F.Cu")
+		(net "+3.3V")
+	)
+	(segment
 		(start 111.4 66.85)
 		(end 111.025 66.85)
@@
 	)
 	(segment
-		(start 106.75 68.75)
-		(end 107 68.5)
-		(width 0.3)
-		(layer "F.Cu")
-		(net "GND")
-	)
-	(segment
 		(start 116.225 67.275)
 		(end 117 66.5)
@@
 	)
 	(segment
-		(start 119 88)
-		(end 118 89)
+		(start 102.43 68.75)
+		(end 103.75 68.75)
 		(width 0.5)
 		(layer "F.Cu")
@@
 	)
 	(segment
-		(start 111.4 66.2)
-		(end 110.7 66.2)
-		(width 0.3)
+		(start 119 88)
+		(end 118 89)
+		(width 0.5)
 		(layer "F.Cu")
 		(net "GND")
 	)
 	(segment
-		(start 105.43 68.75)
-		(end 106.75 68.75)
+		(start 111.4 66.2)
+		(end 110.7 66.2)
 		(width 0.3)
 		(layer "F.Cu")
@@
 	)
 	(segment
+		(start 128.705 66)
+		(end 128.705 64.155)
+		(width 0.5)
+		(layer "F.Cu")
+		(net "GND")
+	)
+	(segment
 		(start 139.15 80.3)
 		(end 140.8 80.3)
@@
 	)
 	(segment
-		(start 128.705 66.655)
-		(end 128.705 68.295)
-		(width 0.5)
-		(layer "F.Cu")
-		(net "GND")
-	)
-	(segment
 		(start 140.8 80.3)
 		(end 141 80.5)
@@
 	)
 	(segment
-		(start 116.775 70.5)
-		(end 118 70.5)
+		(start 103.75 68.75)
+		(end 104 68.5)
 		(width 0.5)
 		(layer "F.Cu")
@@
 	)
 	(segment
-		(start 128.705 68.295)
-		(end 128.5 68.5)
+		(start 116.775 70.5)
+		(end 118 70.5)
 		(width 0.5)
 		(layer "F.Cu")
@@
 	)
 	(via
+		(at 104 68.5)
+		(size 0.7)
+		(drill 0.3)
+		(layers "F.Cu" "B.Cu")
+		(net "GND")
+	)
+	(via
 		(at 101 77)
 		(size 0.6)
@@
 	)
 	(via
-		(at 128.5 68.5)
+		(at 128.705 66)
 		(size 0.6)
 		(drill 0.3)
@@
 	)
 	(segment
-		(start 136.325 71.675)
-		(end 137.475 71.675)
-		(width 0.5)
+		(start 138.6 75.15)
+		(end 139.15 75.7)
+		(width 0.3)
 		(layer "F.Cu")
 		(net "VBUS")
 	)
 	(segment
-		(start 138.6 75.15)
-		(end 139.15 75.7)
-		(width 0.3)
+		(start 131.305 64.155)
+		(end 131.305 66.655)
+		(width 0.5)
 		(layer "F.Cu")
 		(net "VBUS")
@@
 	)
 	(segment
+		(start 131.305 66.655)
+		(end 136.325 71.675)
+		(width 0.5)
+		(layer "F.Cu")
+		(net "VBUS")
+	)
+	(segment
 		(start 141.7 95.3)
 		(end 135.5 101.5)
@@
 	)
 	(segment
-		(start 131.305 66.655)
+		(start 137.475 71.675)
 		(end 136.325 71.675)
 		(width 0.5)
@@
 	)
 	(segment
-		(start 137.475 71.675)
-		(end 138.6 72.8)
+		(start 138.6 72.8)
+		(end 137.475 71.675)
 		(width 0.5)
 		(layer "F.Cu")
@@
 	)
 	(segment
-		(start 130.555 67.730001)
-		(end 130.655 67.630001)
+		(start 130.555 65.230001)
+		(end 130.655 65.130001)
 		(width 0.2)
 		(layer "F.Cu")
@@
 	)
 	(segment
-		(start 130.555 76.763198)
-		(end 130.555 67.730001)
+		(start 130.655 65.130001)
+		(end 130.655 64.155)
 		(width 0.2)
 		(layer "F.Cu")
@@
 	)
 	(segment
-		(start 124.35 77.75)
-		(end 125.512501 77.75)
+		(start 129.593198 77.725)
+		(end 130.555 76.763198)
 		(width 0.2)
 		(layer "F.Cu")
@@
 	)
 	(segment
-		(start 125.512501 77.75)
-		(end 125.537501 77.725)
+		(start 125.537501 77.725)
+		(end 129.593198 77.725)
 		(width 0.2)
 		(layer "F.Cu")
@@
 	)
 	(segment
-		(start 129.593198 77.725)
-		(end 130.555 76.763198)
+		(start 130.555 76.763198)
+		(end 130.555 65.230001)
 		(width 0.2)
 		(layer "F.Cu")
@@
 	)
 	(segment
-		(start 125.537501 77.725)
-		(end 129.593198 77.725)
+		(start 125.512501 77.75)
+		(end 125.537501 77.725)
 		(width 0.2)
 		(layer "F.Cu")
@@
 	)
 	(segment
-		(start 130.655 67.630001)
-		(end 130.655 66.655)
+		(start 124.35 77.75)
+		(end 125.512501 77.75)
 		(width 0.2)
 		(layer "F.Cu")
@@
 	)
 	(segment
-		(start 130.105 67.730001)
-		(end 130.005 67.630001)
+		(start 125.512501 77.25)
+		(end 125.537501 77.275)
 		(width 0.2)
 		(layer "F.Cu")
@@
 	)
 	(segment
-		(start 125.537501 77.275)
-		(end 129.406802 77.275)
+		(start 130.105 76.576802)
+		(end 130.105 65.230001)
 		(width 0.2)
 		(layer "F.Cu")
@@
 	)
 	(segment
-		(start 130.105 76.576802)
-		(end 130.105 67.730001)
+		(start 125.537501 77.275)
+		(end 129.406802 77.275)
 		(width 0.2)
 		(layer "F.Cu")
@@
 	)
 	(segment
-		(start 124.35 77.25)
-		(end 125.512501 77.25)
+		(start 130.005 65.130001)
+		(end 130.005 64.155)
 		(width 0.2)
 		(layer "F.Cu")
@@
 	)
 	(segment
-		(start 130.005 67.630001)
-		(end 130.005 66.655)
+		(start 130.105 65.230001)
+		(end 130.005 65.130001)
 		(width 0.2)
 		(layer "F.Cu")
@@
 	)
 	(segment
-		(start 125.512501 77.25)
-		(end 125.537501 77.275)
+		(start 124.35 77.25)
+		(end 125.512501 77.25)
 		(width 0.2)
 		(layer "F.Cu")
@@
 	)
 	(segment
+		(start 106.5925 70.5875)
+		(end 105.43 71.75)
+		(width 0.3)
+		(layer "F.Cu")
+		(net "Net-(SW1-B)")
+	)
+	(segment
 		(start 110 70.5875)
 		(end 106.5925 70.5875)
@@
 	)
 	(segment
-		(start 106.5925 70.5875)
-		(end 105.43 71.75)
+		(start 105.43 71.75)
+		(end 102.43 71.75)
 		(width 0.3)
 		(layer "F.Cu")
