File: KiCad/flight_controller_pcb.kicad_sch (KiCad schematic)
At the start: 47 parts, among them J1 USB_B, J13 Conn_01x02_Pin, J2 Conn_01x04_Pin, SW1 SW_SPDT, SW3 SW_Push, U1 STM32F405RGTx, U2 LM2596S-5, U3 AMS1117-3.3, U4 ICM-20602, U5 BMP280, Y1 16Mhz

Commit message: Improve project documentation and structure
Parts:
- removed C16, C17: 22u, Capacitor_SMD:C_1206_3216Metric, symbol Device:C
- removed D1, D2, D3: 1N5822, Diode_THT:D_DO-201AD_P15.24mm_Horizontal, symbol Diode:1N5822
- removed J1: USB_B, Connector_USB:USB_Micro-AB_Molex_47590-0001, symbol Connector:USB_B
- removed J13: Conn_01x02_Pin, Connector_Wire:SolderWire-2.5sqmm_1x02_P7.2mm_D2.4mm_OD3.6mm, symbol Connector:Conn_01x02_Pin
- removed L1: 33u, Inductor_SMD:L_1210_3225Metric_Pad1.42x2.65mm_HandSolder, symbol Device:L
- removed SW3: SW_Push, Button_Switch_THT:SW_PUSH_6mm, symbol Switch:SW_Push
- removed U2: LM2596S-5, Package_TO_SOT_SMD:TO-263-5_TabPin3, symbol Regulator_Switching:LM2596S-5
- removed U3: AMS1117-3.3, Package_TO_SOT_SMD:SOT-223-3_TabPin2, symbol Regulator_Linear:AMS1117-3.3
- added J3, J4, J5, J6: Conn_01x03_Pin, Connector_PinHeader_2.54mm:PinHeader_1x03_P2.54mm_Vertical, symbol Connector:Conn_01x03_Pin
- added J7: USB3_B_Micro, Connector_USB:USB_Micro-B_Wuerth_629105150521, symbol Connector:USB3_B_Micro
- added R4: 1k5, Resistor_SMD:R_0402_1005Metric, symbol Device:R
- added U2: AMS1117-3.3, Package_TO_SOT_SMD:SOT-223-3_TabPin2, symbol Regulator_Linear:AMS1117-3.3
- C14: value 680u -> 22u; footprint Capacitor_THT:C_Radial_D10.0mm_H12.5mm_P5.00mm -> Capacitor_SMD:C_0805_2012Metric
- C15: value 220u -> 22u; footprint Capacitor_THT:C_Radial_D10.0mm_H12.5mm_P5.00mm -> Capacitor_SMD:C_0805_2012Metric
- H1, H2, H3, H4: footprint MountingHole:MountingHole_2.5mm_Pad_Via -> MountingHole:MountingHole_2.1mm
Connections:
- net 5V_DC is gone; now on net GND: C15.2
- net +3.3V: now also C15.1, U4.5 (~{CS}), U2.2 (VO)
- net ESC1: now also J3.1 (Pin_1)
- net ESC2: now also J4.1 (Pin_1)
- net ESC3: now also J6.1 (Pin_1)
- net ESC4: now also J5.1 (Pin_1)
- net GND: now also SW1.1 (A), U4.4 (SAO/SD0), J3.3 (Pin_3), J4.3 (Pin_3), J5.3 (Pin_3), J6.3 (Pin_3), J7.5 (GND), U2.1 (GND); no longer C15.1, R1.2
- net SCL: now also U4.2 (SCL/SPC)
- net SDA: now also U4.3 (SDA/SDI)
- net USB_D-: now reaches U1.44 (PA11)
- net USB_D-: now also J7.2 (D-)
- net USB_D+: now reaches U1.45 (PA12)
- net USB_D+: now also J7.3 (D+), R4.2
- net at U1.21 (PA5): no longer U4.2 (SCL/SPC)
- net at U1.22 (PA6): no longer U4.4 (SAO/SD0)
- net at U1.23 (PA7): no longer U4.3 (SDA/SDI)
- net at U1.26 (PB0): no longer U4.5 (~{CS})
- net at U1.27 (PB1): no longer U4.6 (INT)
- net at SW1.2 (B): now also R1.1; no longer U1.60 (BOOT0)
- net ADC1_PIN: no longer names the net of U1.20 (PA4)
- net ESC5: no longer names the net of U1.58 (PB6)
- net ESC6: no longer names the net of U1.59 (PB7)
- net LIPO_BAT renamed VBUS
- net VBUS: now also J3.2 (Pin_2), J7.1 (VBUS), U2.3 (VI)
- net UART4_RX: no longer names the net of U1.52 (PC11)
- net UART4_TX: no longer names the net of U1.51 (PC10)
- net USART1_RX: no longer names the net of U1.43 (PA10)
- new net: R1.2, U1.60 (BOOT0)
- new net +3V3: R4.1
- no-connect marks 29 -> 49
Other:
- removed sheet Second_controller
- note removed: "3.3 LDO Regulator"
- note removed: "5v buck covertor"
- note removed: "Regulated Dc output(5V)"
- note removed: "Unregulated Dc input"
- moved on the sheet: C18, C19, C20, C21, C22, C23, H1, H2, H3, H4, U4, U5
